File: Gametroller/hardware/gametroller.sch (EAGLE design)
At the start: 46 parts, among them J1 microUSB, J2 PJ-002AH-SMT-TR, J3 USB-A, SW1 SPST_TACT-KMR2, U1 LP5907MFX-3.3/NOPB, U16 AOZ1280CI, U2 TPS2115AIPWRQ1-SON8, U4 ATSAMD21G18_QFN, X2 32.768

Commit message: Minor changes to PCB
* Added "power good" LED to 3V3 rail
* Removed silkscreen text for part numbers (just not enough room)
* Increased voltage output on 5V step-down converter
* Added silkscreen text for pin numbers
Parts:
- added D1: RED, gametroller:LED0805_NOOUTLINE
- added R3: 1k, gametroller:R-US_R0603
- R1: value 51k -> 56k
Connections:
- new net N$3: D1.A, R3.2
- net +3V3: now also R3.1
- net GND: now also D1.C
Other:
- moved on the sheet: D4, D5, R2, R7
